Commit message: Pick completo

File: src/piper_celda_description/urdf/piper_x.gazebo.xacro (robot description, xacro)
@@ -28,11 +28,7 @@
       <xacro:joint_pos jname="${prefix}joint6" lmin="-3.14"   lmax="3.14"/>
       <xacro:joint_pos jname="${prefix}joint7" lmin="0.0"     lmax="0.035"/>
-      <!-- joint8 no se comanda: sigue a joint7 por el <mimic> del URDF -->
-      <joint name="${prefix}joint8">
-        <param name="mimic">${prefix}joint7</param>
-        <param name="multiplier">-1</param>
-        <state_interface name="position"/>
-        <state_interface name="velocity"/>
-      </joint>
+      <!-- joint8 se comanda igual que joint7, con signo contrario. El
+           controlador manda los dos a la vez. -->
+      <xacro:joint_pos jname="${prefix}joint8" lmin="-0.035" lmax="0.0"/>
     </ros2_control>
     <!-- ============ plugin del simulador ============ -->

File: src/piper_celda_description/urdf/piper_x.urdf.xacro (robot description, xacro)
@@ -5,5 +5,5 @@
        - Link7 tenia mass=0 e inercia nula: se le asigno la masa/inercia de Link8.
        - Colisiones de base_link..Link6 sustituidas por cascos convexos (STL).
-       - joint8 declarado como mimic de joint7 (pinza de un solo grado de libertad).
+       - joint8 comandado explicitamente en espejo de joint7, sin <mimic>.
        - Anadido ros2_control + plugin gz_ros2_control para Gazebo Harmonic. -->
 <robot xmlns:xacro="http://www.ros.org/wiki/xacro" name="piper_x">
@@ -191,7 +191,13 @@
     <axis xyz="0 0 -1"/>
     <limit lower="0" upper="0.035" effort="60" velocity="0.5"/>
-    <dynamics damping="10.0" friction="1.0"/>
-  </joint>
-  <!-- Dedo espejo: la pinza tiene un solo grado de libertad real -->
+    <!-- Amortiguamiento y friccion bajos. Con damping=10 y friction=1 el dedo,
+         que pesa 26 g, no llegaba a moverse y el controlador abortaba con
+         violacion de tolerancia de trayectoria. -->
+    <dynamics damping="0.5" friction="0.05"/>
+  </joint>
+  <!-- Dedo espejo. Se comanda EXPLICITAMENTE, sin <mimic>: en Jazzy,
+       ros2_control ya lee los mimic del URDF por su cuenta, y declararlos
+       ademas en el bloque ros2_control aplica la restriccion dos veces y
+       deja la pinza bloqueada (el comando llega, el dedo no se mueve). -->
   <joint name="${P}joint8" type="prismatic">
     <origin xyz="0 0 0.13503" rpy="-1.5708 0 1.5708"/>
@@ -199,6 +205,5 @@
     <axis xyz="0 0 1"/>
     <limit lower="-0.035" upper="0" effort="60" velocity="0.5"/>
-    <mimic joint="${P}joint7" multiplier="-1" offset="0"/>
-    <dynamics damping="10.0" friction="1.0"/>
+    <dynamics damping="0.5" friction="0.05"/>
   </joint>
   <joint name="${P}joint_tcp" type="fixed">
